File: COVID-19 Test SAO/KiCad/drawing.kicad_pcb (KiCad board)
At the start: 2 copper layers, 16 x 50 mm, 12 parts, among them J1 Conn_02x03_Odd_Even, U1 NE555D

Commit message: moved labels, gerber version 3 for HiP.berlin
Parts:
- moved Ref** 27.8 mm to (4.90, -5.00)
Other:
- board text added: "2022/11"
- board text added: "@davedarko@chaos.social"
- board text added: "C1+R2 main blink parts R3 for constant LED R4 for blinking LED"
- board text added: "https://hackaday.io/project/187615"
- board text removed: "2022/09"
- board text removed: "@davedarko"
- board text removed: "JLCJLCJLCJLC"
Changed lines of the file:
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@@
     (property "Sheetname" "")
     (attr smd)
-    (fp_text reference "R4" (at 0 -1.651 -90) (layer "B.SilkS")
+    (fp_text reference "R4" (at 2.656 -0.039) (layer "B.SilkS")
       (effects (font (size 1 1) (thickness 0.15)) (justify mirror))
     )
@@
     (fp_line (start 1 -0.625) (end -1 -0.625) (layer "B.Fab") (width 0.1))
     (fp_line (start -1 -0.625) (end -1 0.625) (layer "B.Fab") (width 0.1))
-    (pad "1" smd roundrect locked (at -1 0 270) (size 1.2 1.4) (layers "B.Cu" "B.Paste" "B.Mask") (roundrect_rratio 0.208333)
+    (pad "1" smd roundrect locked (at -1 0 270) (size 1.2 1.4) (layers "B.Cu" "B.Paste" "B.Mask") (roundrect_rratio 0.2083333333)
       (net 12 "Net-(R4-Pad1)") (pintype "passive"))
-    (pad "2" smd roundrect locked (at 1 0 270) (size 1.2 1.4) (layers "B.Cu" "B.Paste" "B.Mask") (roundrect_rratio 0.208333)
+    (pad "2" smd roundrect locked (at 1 0 270) (size 1.2 1.4) (layers "B.Cu" "B.Paste" "B.Mask") (roundrect_rratio 0.2083333333)
       (net 9 "Net-(D2-Pad2)") (pintype "passive"))
     (model "${KISYS3DMOD}/Resistor_SMD.3dshapes/R_0805_2012Metric.wrl"
@@
     (property "Sheetname" "")
     (attr smd)
-    (fp_text reference "R3" (at 0 -1.524 270) (layer "B.SilkS")
+    (fp_text reference "R3" (at 2.524 -0.012) (layer "B.SilkS")
       (effects (font (size 1 1) (thickness 0.15)) (justify mirror))
     )
@@
     (fp_line (start -1 0.625) (end 1 0.625) (layer "B.Fab") (width 0.1))
     (fp_line (start 1 0.625) (end 1 -0.625) (layer "B.Fab") (width 0.1))
-    (pad "1" smd roundrect locked (at -1 0 90) (size 1.2 1.4) (layers "B.Cu" "B.Paste" "B.Mask") (roundrect_rratio 0.208333)
+    (pad "1" smd roundrect locked (at -1 0 90) (size 1.2 1.4) (layers "B.Cu" "B.Paste" "B.Mask") (roundrect_rratio 0.2083333333)
       (net 1 "VCC") (pintype "passive"))
-    (pad "2" smd roundrect locked (at 1 0 90) (size 1.2 1.4) (layers "B.Cu" "B.Paste" "B.Mask") (roundrect_rratio 0.208333)
+    (pad "2" smd roundrect locked (at 1 0 90) (size 1.2 1.4) (layers "B.Cu" "B.Paste" "B.Mask") (roundrect_rratio 0.2083333333)
       (net 8 "Net-(D1-Pad2)") (pintype "passive"))
     (model "${KISYS3DMOD}/Resistor_SMD.3dshapes/R_0805_2012Metric.wrl"
@@
     (property "Sheetname" "")
     (attr smd)
-    (fp_text reference "C1" (at 0 1.68 90) (layer "B.SilkS")
+    (fp_text reference "C1" (at 2.588 0.039 180) (layer "B.SilkS")
       (effects (font (size 1 1) (thickness 0.15)) (justify mirror))
     )
@@
     (fp_line (start 1 0.625) (end 1 -0.625) (layer "B.Fab") (width 0.1))
     (fp_line (start -1 -0.625) (end -1 0.625) (layer "B.Fab") (width 0.1))
-    (pad "1" smd roundrect locked (at -1.0375 0 90) (size 1.175 1.45) (layers "B.Cu" "B.Paste" "B.Mask") (roundrect_rratio 0.212766)
+    (pad "1" smd roundrect locked (at -1.0375 0 90) (size 1.175 1.45) (layers "B.Cu" "B.Paste" "B.Mask") (roundrect_rratio 0.2127659574)
       (net 11 "Net-(C1-Pad1)") (pintype "passive"))
-    (pad "2" smd roundrect locked (at 1.0375 0 90) (size 1.175 1.45) (layers "B.Cu" "B.Paste" "B.Mask") (roundrect_rratio 0.212766)
+    (pad "2" smd roundrect locked (at 1.0375 0 90) (size 1.175 1.45) (layers "B.Cu" "B.Paste" "B.Mask") (roundrect_rratio 0.2127659574)
       (net 4 "GND") (pintype "passive"))
     (model "${KISYS3DMOD}/Capacitor_SMD.3dshapes/C_0805_2012Metric.wrl"
@@
     (property "Sheetname" "")
     (attr smd)
-    (fp_text reference "R1" (at 0 1.524 -90) (layer "B.SilkS")
+    (fp_text reference "R1" (at 2.577 0.012) (layer "B.SilkS")
       (effects (font (size 1 1) (thickness 0.15)) (justify mirror))
     )
@@
     (fp_line (start -1 0.625) (end 1 0.625) (layer "B.Fab") (width 0.1))
     (fp_line (start -1 -0.625) (end -1 0.625) (layer "B.Fab") (width 0.1))
-    (pad "1" smd roundrect locked (at -1 0 270) (size 1.2 1.4) (layers "B.Cu" "B.Paste" "B.Mask") (roundrect_rratio 0.208333)
+    (pad "1" smd roundrect locked (at -1 0 270) (size 1.2 1.4) (layers "B.Cu" "B.Paste" "B.Mask") (roundrect_rratio 0.2083333333)
       (net 1 "VCC") (pintype "passive"))
-    (pad "2" smd roundrect locked (at 1 0 270) (size 1.2 1.4) (layers "B.Cu" "B.Paste" "B.Mask") (roundrect_rratio 0.208333)
+    (pad "2" smd roundrect locked (at 1 0 270) (size 1.2 1.4) (layers "B.Cu" "B.Paste" "B.Mask") (roundrect_rratio 0.2083333333)
       (net 10 "Net-(R1-Pad2)") (pintype "passive"))
     (model "${KISYS3DMOD}/Resistor_SMD.3dshapes/R_0805_2012Metric.wrl"
@@
     (fp_line (start -1 0.3) (end -1 -0.6) (layer "B.Fab") (width 0.1))
     (fp_line (start -0.7 0.6) (end -1 0.3) (layer "B.Fab") (width 0.1))
-    (pad "1" smd roundrect locked (at -1.025 0 270) (size 1.15 1.4) (layers "B.Cu" "B.Paste" "B.Mask") (roundrect_rratio 0.217391)
+    (pad "1" smd roundrect locked (at -1.025 0 270) (size 1.15 1.4) (layers "B.Cu" "B.Paste" "B.Mask") (roundrect_rratio 0.2173913043)
       (net 4 "GND") (pinfunction "K") (pintype "passive"))
-    (pad "2" smd roundrect locked (at 1.025 0 270) (size 1.15 1.4) (layers "B.Cu" "B.Paste" "B.Mask") (roundrect_rratio 0.217391)
+    (pad "2" smd roundrect locked (at 1.025 0 270) (size 1.15 1.4) (layers "B.Cu" "B.Paste" "B.Mask") (roundrect_rratio 0.2173913043)
       (net 9 "Net-(D2-Pad2)") (pinfunction "A") (pintype "passive"))
     (model "${KISYS3DMOD}/LED_SMD.3dshapes/LED_0805_2012Metric.wrl"
@@
     (fp_line (start 4.52 -8.99) (end -1.98 -8.99) (layer "B.Fab") (width 0.1))
     (fp_line (start -1.98 -4.59) (end -1.98 -4.59) (layer "B.Fab") (width 0.1))
-    (pad "1" thru_hole roundrect locked (at 0 0 270) (size 1.7 1.7) (drill 1) (layers *.Cu *.Mask) (roundrect_rratio 0.147059)
+    (pad "1" thru_hole roundrect locked (at 0 0 270) (size 1.7 1.7) (drill 1) (layers *.Cu *.Mask) (roundrect_rratio 0.1470588235)
       (net 1 "VCC") (pinfunction "Pin_1") (pintype "passive"))
     (pad "2" thru_hole circle locked (at 2.54 0 270) (size 1.7 1.7) (drill 1) (layers *.Cu *.Mask)
@@
     (property "Sheetname" "")
     (attr smd)
-    (fp_text reference "R2" (at 0 1.65 90) (layer "B.SilkS")
+    (fp_text reference "R2" (at 2.597 -0.088 180) (layer "B.SilkS")
       (effects (font (size 1 1) (thickness 0.15)) (justify mirror))
     )
@@
     (fp_line (start -1 0.625) (end 1 0.625) (layer "B.Fab") (width 0.1))
     (fp_line (start -1 -0.625) (end -1 0.625) (layer "B.Fab") (width 0.1))
-    (pad "1" smd roundrect locked (at -1 0 270) (size 1.2 1.4) (layers "B.Cu" "B.Paste" "B.Mask") (roundrect_rratio 0.208333)
+    (pad "1" smd roundrect locked (at -1 0 270) (size 1.2 1.4) (layers "B.Cu" "B.Paste" "B.Mask") (roundrect_rratio 0.2083333333)
       (net 10 "Net-(R1-Pad2)") (pintype "passive"))
-    (pad "2" smd roundrect locked (at 1 0 270) (size 1.2 1.4) (layers "B.Cu" "B.Paste" "B.Mask") (roundrect_rratio 0.208333)
+    (pad "2" smd roundrect locked (at 1 0 270) (size 1.2 1.4) (layers "B.Cu" "B.Paste" "B.Mask") (roundrect_rratio 0.2083333333)
       (net 11 "Net-(C1-Pad1)") (pintype "passive"))
     (model "${KISYS3DMOD}/Resistor_SMD.3dshapes/R_0805_2012Metric.wrl"
@@
     (fp_line (start -0.7 0.6) (end -1 0.3) (layer "B.Fab") (width 0.1))
     (fp_line (start -1 -0.6) (end 1 -0.6) (layer "B.Fab") (width 0.1))
-    (pad "1" smd roundrect locked (at -1.025 0 270) (size 1.15 1.4) (layers "B.Cu" "B.Paste" "B.Mask") (roundrect_rratio 0.217391)
+    (pad "1" smd roundrect locked (at -1.025 0 270) (size 1.15 1.4) (layers "B.Cu" "B.Paste" "B.Mask") (roundrect_rratio 0.2173913043)
       (net 4 "GND") (pinfunction "K") (pintype "passive"))
-    (pad "2" smd roundrect locked (at 1.025 0 270) (size 1.15 1.4) (layers "B.Cu" "B.Paste" "B.Mask") (roundrect_rratio 0.217391)
+    (pad "2" smd roundrect locked (at 1.025 0 270) (size 1.15 1.4) (layers "B.Cu" "B.Paste" "B.Mask") (roundrect_rratio 0.2173913043)
       (net 8 "Net-(D1-Pad2)") (pinfunction "A") (pintype "passive"))
     (model "${KISYS3DMOD}/LED_SMD.3dshapes/LED_0805_2012Metric.wrl"
@@
   )
   (footprint "kicad footprints:davedarko_logo_silk_ext" (layer "B.Cu")
-    (at -5 21 180)
+    (at 4.9 -5 180)
     (attr through_hole)
     (fp_text reference "Ref**" (at 0 0) (layer "B.SilkS") hide
@@
   (gr_line locked (start 8 -23) (end 8 23) (layer "Edge.Cuts") (width 0.15))
   (gr_arc locked (start 6 -25) (mid 7.414214 -24.414214) (end 8 -23) (layer "Edge.Cuts") (width 0.15))
-  (gr_text "@davedarko" (at 0 -23.114) (layer "B.SilkS")
+  (gr_text "C1+R2 main blink parts\nR3 for constant LED\nR4 for blinking LED\n" (at 7.4 22.2) (layer "B.SilkS")
+    (effects (font (size 0.8 0.8) (thickness 0.12)) (justify left mirror))
+  )
+  (gr_text "@davedarko@chaos.social" (at 0 -20.8) (layer "B.SilkS")
+    (effects (font (size 0.8 0.8) (thickness 0.12)) (justify mirror))
+  )
+  (gr_text "https://hackaday.io/project/187615" (at -7.2 14.7 270) (layer "B.SilkS")
+    (effects (font (size 0.8 0.8) (thickness 0.12)) (justify left mirror))
+  )
+  (gr_text "2022/11" (at 0 -22.9) (layer "B.SilkS")
     (effects (font (size 1.5 1.5) (thickness 0.3)) (justify mirror))
   )
-  (gr_text "JLCJLCJLCJLC" (at 6.223 -7.493 90) (layer "B.SilkS")
-    (effects (font (size 1.5 1.5) (thickness 0.3)) (justify mirror))
-  )
-  (gr_text "2022/09" (at 0 -20.828) (layer "B.SilkS")
-    (effects (font (size 1.5 1.5) (thickness 0.3)) (justify mirror))
-  )
