File: HelloMyNameIs/henlo_blinkyparts_style/henlo_blinkyparts_style.kicad_pcb (KiCad board)
At the start: 2 copper layers, 40 x 34 mm, 6 parts, among them J1 Conn_02x03_Odd_Even

Commit message: added 2 more and updated solo
Routing:
- net GND: vias 0 -> 2
Changed lines of the file:
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@@
 		(net 5)
+	)
+	(via
+		(at 38.8 30.9)
+		(size 0.6)
+		(drill 0.3)
+		(layers "F.Cu" "B.Cu")
+		(free yes)
+		(net 6)
+	)
+	(via
+		(at 37.9 32.5)
+		(size 0.6)
+		(drill 0.3)
+		(layers "F.Cu" "B.Cu")
+		(free yes)
+		(net 6)
 	)
 	(zone
