File: SAO library stick/SAO_library.kicad_sch (KiCad schematic)
At the start: 55 parts

Commit message: Added more designs and updates
Parts:
- C1, C10, C11, C12, C13, C14, C15, C16, C17, C18, C19, C2, C20, C3, C4, C5, C6, C7, C8, C9: value (none) -> C; footprint (none) -> Capacitor_SMD:C_1206_3216Metric_Pad1.33x1.80mm_HandSolder
- D1, D2: value (none) -> LED; footprint (none) -> LED_SMD:LED_1206_3216Metric
- H1, H2, H3, H4, H5, H6, H7, H8: value (none) -> MountingHole; footprint (none) -> MountingHole:MountingHole_3.2mm_M3_Pad_Via
- J1: value (none) -> Barrel_Jack_Switch; footprint (none) -> Connector_BarrelJack:BarrelJack_CUI_PJ-102AH_Horizontal
- J2, J3: value (none) -> Conn_01x04_Female; footprint (none) -> Connector_JST:JST_SH_SM04B-SRSS-TB_1x04-1MP_P1.00mm_Horizontal
- JP1, JP2: value (none) -> Jumper_NO_Small; footprint (none) -> Jumper:SolderJumper-2_P1.3mm_Open_RoundedPad1.0x1.5mm
- R1, R2: value (none) -> R; footprint (none) -> Resistor_SMD:R_1206_3216Metric_Pad1.30x1.75mm_HandSolder
- U1, U18: value (none) -> AMS1117-3.3; footprint (none) -> Package_TO_SOT_SMD:SOT-223-3_TabPin2
- U10, U11, U12, U13, U14, U15, U16, U17, U2, U3, U4, U5, U6, U7, U8, U9: value (none) -> SAOV1.69BIS; footprint (none) -> Connector_PinSocket_2.54mm:PinSocket_2x03_P2.54mm_Vertical
