File: SoloCarbonite/SoloCarbonite/SoloCarbonite.kicad_pcb (KiCad board)
At the start: 2 copper layers, 27 x 67 mm, 21 parts, among them J1 Conn_02x03_Odd_Even, J2 Conn_01x04_Socket, U1 ATtiny412-SS

Commit message: Added more designs and updates
Parts:
- removed J2: Conn_01x04_Socket, Connector_JST:JST_SH_SM04B-SRSS-TB_1x04-1MP_P1.00mm_Horizontal
- removed Ref**: Val**, davedarko:davedarko_logo_silk_outline
- removed TP2, TP3: TestPoint, TestPoint:TestPoint_Pad_D2.0mm
- added BT1: Battery, SAOAO:Battery_holder_CR2023_BS-08-B2, B.Cu at (13.1, 37.0)
- added SW1: SW_SPDT, Button_Switch_SMD:SW_SPDT_PCM12, B.Cu at (24.5, 58.5)
- added TP4: TestPoint, TestPoint:TestPoint_Pad_D3.0mm, B.Cu at (13.5, 2.35)
- moved D1 132.3 mm to (21.4, 50.4)
- moved R2 132.1 mm to (5.50, 57.7)
- moved C3 132.1 mm to (18.9, 21.1), turned to 90 degrees
- moved R1 131.3 mm to (5.40, 59.5)
- moved C2 131.1 mm to (19.4, 17.0)
- moved D2 131.1 mm to (21.4, 21.0)
- moved J1 131.1 mm to (11.1, 62.8)
- moved D3 131.1 mm to (21.4, 13.0)
- moved D4 131.1 mm to (21.4, 4.85)
- moved TP1 131.1 mm to (12.5, 14.1)
- moved C1 131.0 mm to (19.0, 9.95)
- moved C5 130.9 mm to (15.5, 10.00)
- moved D5 130.3 mm to (12.9, 9.95)
- moved JP2 125.2 mm to (19.6, 64.3)
- moved JP1 123.2 mm to (19.6, 60.1)
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Connections:
- J1 pad 1: VCC -> Net-(J1-Pin_1)
- U1 pad 3: Net-(U1-PA7) -> unconnected-(U1-PA7-Pad3)
- U1 pad 7: Net-(U1-PA3) -> unconnected-(U1-PA3-Pad7)
Routing:
- net VCC: track 171.1 -> 122.5 mm
- net SCL: track 55.1 -> 11.9 mm, vias 1 -> 0
- net SDA: track 43.2 -> 14.4 mm, vias 1 -> 0
- net Net-(BT1-+): track 0.00 -> 15.7 mm
- net Net-(J1-Pin_1): track 0.00 -> 15.2 mm, vias 0 -> 1
- net Net-(D1-DIN): track 7.77 -> 20.1 mm
- net UPDI: track 16.3 -> 8.62 mm
- net Net-(J1-Pin_6): track 14.1 -> 8.74 mm
- net Net-(U1-PA3): track 5.28 -> 0.00 mm
- net GND: track 10.3 -> 15.1 mm, vias 24 -> 5
- net Net-(D1-DOUT): track 30.6 -> 26.4 mm
- net Net-(JP2-A): track 16.1 -> 11.9 mm
- net Net-(J1-Pin_5): track 9.52 -> 5.76 mm
- net Net-(U1-PA7): track 3.56 -> 0.00 mm
- net Net-(D5-DOUT): track 5.26 -> 2.56 mm
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Other:
- board text removed: "CUT UPDI FROM GPIO2"
- board text removed: "GND"
- board text removed: "GPIO1"
- board text removed: "GPIO2"
- board text removed: "PA3"
- board text removed: "PA7"
- board text removed: "QWIIC"
- board text removed: "SCL"
- board text removed: "SDA"
- board text removed: "VCC"
