File: SoloCarbonite/SoloCarbonite/SoloCarbonite.kicad_sch (KiCad schematic)
At the start: 12 parts, among them J1 Conn_02x03_Odd_Even, U1 ATtiny202-SS

Commit message: added 2 more and updated solo
Parts:
- removed D1, D2, D3, D4: SK6805, footprint_lib:LED_SK6805-EC3210R, symbol LED:SK6805
- removed U1: ATtiny202-SS, Package_SO:SOIC-8_3.9x4.9mm_P1.27mm, symbol MCU_Microchip_ATtiny:ATtiny202-SS
- added C5: 100nF, Capacitor_SMD:C_0603_1608Metric_Pad1.08x0.95mm_HandSolder, symbol Device:C
- added D1, D2, D3, D4, D5: SK6805-EC3210R, footprint_lib:LED_SK6805-EC3210R, symbol SK6805-EC3210R:SK6805-EC3210R
- added J2: Conn_01x04_Socket, Connector_JST:JST_SH_SM04B-SRSS-TB_1x04-1MP_P1.00mm_Horizontal, symbol Connector:Conn_01x04_Socket
- added JP1: Jumper_2_Bridged, Jumper:SolderJumper-2_P1.3mm_Bridged_RoundedPad1.0x1.5mm, symbol Jumper:Jumper_2_Bridged
- added R1, R2: 10k, Resistor_SMD:R_0603_1608Metric_Pad0.98x0.95mm_HandSolder, symbol Device:R
- added TP2, TP3: TestPoint, TestPoint:TestPoint_Pad_D2.0mm, symbol Connector:TestPoint
- added U1: ATtiny412-SS, Package_SO:SOIC-8_3.9x4.9mm_P1.27mm, symbol MCU_Microchip_ATtiny:ATtiny412-SS
- C1, C2, C3, C4: value C -> 100nF; MPN (none) -> C14663
- J1: footprint Connector_IDC:IDC-Header_2x03_P2.54mm_Vertical -> Connector_PinHeader_2.54mm:PinHeader_2x03_P2.54mm_Vertical; MPN (none) -> DNP
- JP2, TP1: MPN (none) -> DNP
Connections:
- net GND: now also C5.2, D1.1 (VSS), D2.1 (VSS), D3.1 (VSS), D4.1 (VSS), D5.1 (VSS), J2.1 (Pin_1), U1.8 (GND)
- net SCL: now also J2.4 (Pin_4), R1.2, U1.5 (PA2)
- net SDA: now also J2.3 (Pin_3), R2.2, U1.4 (PA1)
- net VCC: now also C5.1, D1.4 (VDD), D2.4 (VDD), D3.4 (VDD), D4.4 (VDD), D5.4 (VDD), J2.2 (Pin_2), R1.1, R2.1, U1.1 (VCC)
- net at TP1.1: now also D5.2 (DOUT)
- net at JP2.2 (C): now also D1.3 (DIN)
- net at J1.6 (Pin_6): now also JP1.2 (B)
- net at JP2.1 (A): now also U1.2 (PA6)
- new net: TP2.1, U1.7 (PA3)
- new net: TP3.1, U1.3 (PA7)
- new net: D3.2 (DOUT), D4.3 (DIN)
- new net: D2.2 (DOUT), D3.3 (DIN)
- new net: D1.2 (DOUT), D2.3 (DIN)
- new net: D4.2 (DOUT), D5.3 (DIN)
- new net UPDI: JP1.1 (A), U1.6 (~{RESET}/PA0)
Other:
- moved on the sheet: TP1

Commit message: Added more designs and updates
Parts:
- removed J2: Conn_01x04_Socket, Connector_JST:JST_SH_SM04B-SRSS-TB_1x04-1MP_P1.00mm_Horizontal, symbol Connector:Conn_01x04_Socket
- removed TP2, TP3: TestPoint, TestPoint:TestPoint_Pad_D2.0mm, symbol Connector:TestPoint
- added BT1: Battery, SAOAO:Battery_holder_CR2023_BS-08-B2, symbol Device:Battery
- added SW1: SW_SPDT, Button_Switch_SMD:SW_SPDT_PCM12, symbol Switch:SW_SPDT
- added TP4: TestPoint, TestPoint:TestPoint_Pad_D3.0mm, symbol Connector:TestPoint
Connections:
- net GND: now also BT1.2 (-), TP4.1
- net VCC: now also SW1.2 (B); no longer J1.1 (Pin_1)
- new net: BT1.1 (+), SW1.1 (A)
- new net: J1.1 (Pin_1), SW1.3 (C)
Other:
- moved on the sheet: JP2
